Commit message: Position of all elements configured

File: ur10e_simple_controller/urdf/ur10e_control.urdf (robot description, URDF)
Before this commit: robot ur10e, 9 links, 8 joints
Joints:
- joint elbow_joint: origin xyz=0.0 -0.1197 0.425 rpy=0.0 0.0 0.0 -> xyz=0.0 -0.123 0.613 rpy=0.0 0.0 0.0
- joint shoulder_lift_joint: origin xyz=0.0 0.13585 0.0 rpy=0.0 1.570796325 0.0 -> xyz=0.0 0.17585 0.0 rpy=0.0 1.570796325 0.0
- joint shoulder_pan_joint: origin xyz=0.0 0.0 0.089159 rpy=0.0 0.0 0.0 -> xyz=0.0 0.0 0.185 rpy=0.0 0.0 0.0
- joint wrist_1_joint: origin xyz=0.0 0.0 0.39225 rpy=0.0 1.570796325 0.0 -> xyz=0.0 0.0 0.57 rpy=0.0 1.570796325 0.0
- joint wrist_2_joint: origin xyz=0.0 0.093 0.0 rpy=0.0 0.0 0.0 -> xyz=0.0 0.135 0.0 rpy=0.0 0.0 0.0
- joint wrist_3_joint: origin xyz=0.0 0.0 0.09465 rpy=0.0 0.0 0.0 -> xyz=0.0 0.0 0.12 rpy=0.0 0.0 0.0
